File: pcb/meter.kicad_sch (KiCad schematic)
At the start: 6 parts, among them U8 INA219AxDCN

Commit message: chore: cleanup
Parts:
- renumbered C34 to C38, C35 to C39, R33 to R40, R34 to R41, R35 to R42, U8 to U10
Changed lines of the file:
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@@
 		(dnp no)
 		(fields_autoplaced yes)
-		(property "Reference" "#PWR035"
+		(property "Reference" "#PWR044"
 			(at 144.78 109.22 0)
 			(effects
@@
 		(dnp no)
 		(fields_autoplaced yes)
-		(property "Reference" "#PWR033"
+		(property "Reference" "#PWR042"
 			(at 144.78 81.28 0)
 			(effects
@@
 		(dnp no)
 		(fields_autoplaced yes)
-		(property "Reference" "R33"
+		(property "Reference" "R40"
 			(at 115.57 85.09 90)
 			(effects
@@
 		(dnp no)
 		(fields_autoplaced yes)
-		(property "Reference" "#PWR034"
+		(property "Reference" "#PWR043"
 			(at 130.81 80.01 0)
 			(effects
@@
 		(dnp no)
 		(fields_autoplaced yes)
-		(property "Reference" "U8"
+		(property "Reference" "U10"
 			(at 146.9741 80.01 0)
 			(effects
@@
 		(on_board yes)
 		(dnp no)
-		(property "Reference" "C35"
+		(property "Reference" "C39"
 			(at 124.46 91.4462 0)
 			(effects
@@
 		(dnp no)
 		(fields_autoplaced yes)
-		(property "Reference" "C34"
+		(property "Reference" "C38"
 			(at 139.7063 73.66 90)
 			(effects
@@
 		(dnp no)
 		(fields_autoplaced yes)
-		(property "Reference" "R34"
+		(property "Reference" "R41"
 			(at 105.41 91.4399 0)
 			(effects
@@
 		(dnp no)
 		(fields_autoplaced yes)
-		(property "Reference" "R35"
+		(property "Reference" "R42"
 			(at 115.57 97.79 90)
 			(effects
