File: pcb/usbc.kicad_sch (KiCad schematic)
At the start: 3 parts, among them J7 ${SHEETNAME}

Commit message: style: replace OTG connector
Parts:
- renumbered J7 to J3
Changed lines of the file:
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@@
 		(dnp no)
 		(fields_autoplaced yes)
-		(property "Reference" "#PWR0101"
+		(property "Reference" "#PWR052"
 			(at 134.62 127 0)
 			(effects
@@
 		(dnp no)
 		(fields_autoplaced yes)
-		(property "Reference" "J7"
+		(property "Reference" "J3"
 			(at 134.62 74.93 0)
 			(effects
